File: aurola-board.brd (EAGLE design)
At the start: 86.4 x 31.8 mm, 84 parts, among them IC1 STM32F051C6T, J1 CONN_PWM, J2 CONN_TEMP, J3 CONN_FAN, J4 CONN_EC11, J5 CONN_I2C, P1 KF128-2P, Q1 600mA/40V, U1 ESP-01F, U2 BL9341, U3 BL9341

Commit message: 输出打样文件
Parts:
- removed R100: 680, standardparts:0805
- added R30: 470, standardparts:0603
- C11: device standardparts:0603 -> standardparts:0805
- C12: value 1uF -> 100nF; device standardparts:0603 -> standardparts:0805
- C13, C14, C15: value 15pF -> 100nF
- C16: value 15pF -> 100uF; device standardparts:0603 -> standardparts:1210
- C17, C20, C21: value 100nF -> 10uF; device standardparts:0603 -> standardparts:1206
- C18: device SparkFun-Capacitors:EIA3216 -> standardparts:1206
- C2: value 100nF -> 15pF; device standardparts:0805 -> standardparts:0603
- C22: value 100uF -> 47UF-POLAR-PANASONIC_D-50V-20%; device standardparts:1210 -> SparkFun-Capacitors:PANASONIC_D
- C23: value 100nF -> 1uF
- C27: value 100nF -> 10uF; device standardparts:0603 -> SparkFun-Capacitors:EIA3216
- C28: value 47UF-POLAR-PANASONIC_D-50V-20% -> 100nF; device SparkFun-Capacitors:PANASONIC_D -> standardparts:0603
- C3, C4, C5: value 10uF -> 15pF; device standardparts:1206 -> standardparts:0603
- C7: device standardparts:0805 -> standardparts:0603
- C8: value 10uF -> 100nF; device standardparts:1206 -> standardparts:0603
- D3: device we-rcl:SMA_DO214AC -> standardparts:0603.LED
- D5: device standardparts:0603.LED -> we-rcl:SMA_DO214AC
- J1: value CONN_PWM -> (none); device conn_smt:PH2.0_8P -> SparkFun-Connectors:1X02
- J2: value CONN_TEMP -> (none); device conn_smt:PH2.0_3P -> SparkFun-Connectors:1X04
- J3: value CONN_FAN -> CONN_PWM; device conn_smt:PH2.0_4P -> conn_smt:PH2.0_8P
- J4: value CONN_EC11 -> TEMP_DO; device conn_smt:PH2.0_4P -> conn_smt:PH2.0_3P
- J5: value CONN_I2C -> CONN_FAN
- J6: value (none) -> CONN_I2C; device SparkFun-Connectors:1X04 -> conn_smt:PH2.0_4P
- J7: value (none) -> EC; device SparkFun-Connectors:1X02 -> conn_smt:PH2.0_4P
- L1: value 10uH -> 10µH; device SparkFun-Coils:CR54 -> SparkFun-Coils:0805
- L3: value 10µH -> 10uH; device SparkFun-Coils:0805 -> SparkFun-Coils:CR54
- R1: value 100k -> 680; device standardparts:0603 -> standardparts:0805
- R10: value 470 -> 14k
- R11, R13: value 470 -> 1k
- R12: value 470 -> 10k
- R14: value 470 -> 33k
- R15: value 4.7k -> 10k
- R19: value 470 -> 4.7k
- R2: value 4.22k -> 560
- R21, R22, R23, R24, R25: value 10k -> 470
- R26: value 4.7k -> 470
- R27: value 560 -> 470
- R28: value 33k -> 470
- R29, R5: value 1k -> 10k
- R3: value 100k -> 10k
- R4: value 13.3k -> 4.7k
- R6: value 14k -> 100k
- R7: value 470 -> 100k
- R8: value 470 -> 13.3k
- R9: value 470 -> 4.22k
- U1: value ESP-01F -> BL9341; device esp_mod:ESP-01F -> dcdc:SOT23-6
- U3: value BL9341 -> ESP-01F; device dcdc:SOT23-6 -> esp_mod:ESP-01F
- Y1: value NX5032CA-8MHZ -> (none)
- Y2: value 32.768KHZ-FC-135 -> (none)
- moved R14 75.1 mm to (83.9, 25.0), turned to 0 degrees
- moved R28 75.1 mm to (10.7, 8.38), turned to 180 degrees
- moved R8 65.9 mm to (74.5, 3.30), turned to 270 degrees
- moved R9 63.1 mm to (72.0, 2.79), turned to 0 degrees
- moved R7 57.8 mm to (68.3, 17.7), turned to 0 degrees
- moved R10 54.5 mm to (65.0, 17.7)
- moved R11 54.5 mm to (64.5, 20.2), turned to 270 degrees
- moved C11 54.4 mm to (73.3, 9.65), turned to 180 degrees
- moved C6 54.1 mm to (15.1, 13.2), turned to 270 degrees
- moved C7 52.9 mm to (21.1, 1.78), turned to 0 degrees
- moved C17 51.3 mm to (65.4, 3.05), turned to 180 degrees
- moved C18 51.2 mm to (67.1, 26.8)
- moved C28 50.4 mm to (31.5, 21.6), turned to 90 degrees
- moved R13 50.0 mm to (59.3, 21.6), turned to 270 degrees
- moved C8 49.8 mm to (23.6, 2.41), turned to 270 degrees
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- renumbered U$1 to Y1, U$2 to Y2
Connections:
- net 12V: now also C18.2, C21.2, D3.P$1, J5.2, L3.P$2, R10.2; no longer C8.2, C9.2, D5.P$1, J3.2, L1.P$2, R6.2
- net 3.3V: now also C15.1, C16.1, C20.2, C23.2, C25.2, C6.2, C7.2, J4.1, J6.1, L1.1, R12.1, R19.1, R2.1, R29.1, R5.1, R8.2, U3.17; no longer C11.2, C12.2, C19.2, C22.1, C23.1, C3.2, C4.2, J2.1, J5.1, L3.1, R22.1, R23.1, R24.1, R25.1, R27.1, R4.2, U1.17
- net EC_A: now also C24.2, J7.3, R16.2; no longer C25.2, J4.3, R25.2
- net EC_B: now also J7.2, R18.2; no longer J4.2, R24.2
- net EC_INT: now also U3.6; no longer U1.6
- net EC_SW: now also C28.2, J7.1, R29.2, U3.10; no longer C27.2, J4.1, R23.2, U1.10
- net FAN_PWM: now also R30.1; no longer R19.1
- net FAN_SPEED: now also J5.3, R20.2; no longer J3.3, R16.2
- net FAN_SW: now also R4.2, U3.8; no longer R26.2, U1.8
- net FLASH: now also J2.2, U3.11; no longer J6.2, U1.11
- net GND: now also C1.1, C15.2, C16.2, C18.1, C22.-, C23.1, C24.1, C27.-, C28.1, C6.1, C8.2, D5.A, J2.1, J4.3, J5.1, J6.4, J7.4, R11.1, R13.1, R14.2, R3.2, R9.1, U3.18, U3.19; no longer C13.1, C14.1, C15.1, C16.1, C18.-, C22.2, C23.2, C24.2, C27.1, C28.-, C8.1, D3.A, J2.3, J3.1, J4.4, J5.4, J6.1, R2.1, R21.2, R28.2, R29.1, R5.1, U1.18, U1.19
- net N$1: now also R7.1, U2.4; no longer R3.1, U3.4
- net N$10: now also J3.2, R22.2; no longer J1.2, R8.2
- net N$11: now also J3.3, R23.2; no longer J1.3, R9.2
- net N$12: now also J3.4, R24.2; no longer J1.4, R12.2
- net N$13: now also J3.5, R25.2; no longer J1.5, R10.2
- net N$14: now also J3.6, R26.2; no longer J1.6, R11.2
- net N$15: now also J3.7, R27.2; no longer J1.7, R13.2
- net N$16: now also J3.8, R28.2; no longer J1.8, R14.2
- net N$17: now also R5.2, U3.4; no longer R20.2, U1.4
- net N$18: now also J5.4, R30.2; no longer J3.4, R19.2
- net N$19: now also R3.1, U3.9; no longer R21.1, U1.9
- net N$2: now also C13.1, U1.6; no longer C1.1, U2.6
- net N$20: now also R4.1; no longer R26.1
- net N$21: now also R1.2; no longer R100.2
- net N$22: now also C1.2, L1.2; no longer C21.2, L3.2
- net N$23: now also U3.7; no longer U1.7
- net N$24: now also R2.2; no longer R27.2
- net N$27: now also R14.1; no longer R28.1
- net N$28: now also D3.P$2, R13.2; no longer D5.P$2, R29.2
- net N$3: now also R6.1, U1.4; no longer R1.1, U2.4
- net N$4: now also R8.1, R9.2, U1.3; no longer R2.2, R4.1, U2.3
- net N$5: now also R10.1, R11.2, U2.3; no longer R5.2, R6.1, U3.3
- net N$6: now also C14.1, L3.P$1, U2.6; no longer C6.1, L1.P$1, U3.6
- net N$7: now also C14.2, U2.1; no longer C6.2, U3.1
- net N$8: now also C13.2, U1.1; no longer C1.2, U2.1
- net N$9: now also J3.1, R21.2; no longer J1.1, R7.2
- net OSC32_IN: now also C4.2; no longer C15.2
- net OSC32_OUT: now also C5.2; no longer C16.2
- net OSC_IN: now also C2.2; no longer C13.2
- net OSC_OUT: now also C3.2; no longer C14.2
- net PWM1: now also R25.1; no longer R10.1
- net PWM2: now also R26.1; no longer R11.1
- net PWM3: now also R27.1; no longer R13.1
- net PWM4: now also R28.1; no longer R14.1
- net PWM5: now also R21.1; no longer R7.1
- net PWM6: now also R22.1; no longer R8.1
- net PWM7: now also R23.1; no longer R9.1
- net PWM8: now also R24.1; no longer R12.1
- net RST: now also C19.2, R12.2, U3.16; no longer C20.2, R22.2, U1.16
- net RX: now also J2.3, U3.14; no longer J6.3, U1.14
- net SCL: now also J6.3, R15.2, U3.13; no longer J5.3, R17.2, U1.13
- net SDA: now also J6.2, R17.2, U3.12; no longer J5.2, R18.2, U1.12
- net SW_CLK: now also J1.2; no longer J7.2
- net SW_DIO: now also J1.1; no longer J7.1
- net TEMP_DO: now also C27.+, J4.2, R19.2; no longer C18.+, J2.2, R15.2
- net TX: now also J2.4, U3.15; no longer J6.4, U1.15
- net VBAT: now also C8.1, R1.1; no longer C24.1, R100.1
- net VIN: now also C11.2, C12.2, C22.+, C9.2, D5.C, R6.2, R7.2, U1.5; no longer C2.2, C28.+, C5.2, C7.2, D3.C, R1.2, R3.2, U3.5
Routing:
- net GND: track 93.6 -> 89.9 mm, vias 79 -> 81
Other:
- board text added: "+"
- board text added: "-"
- board text added: "24V"
