File: aurola-board.brd (EAGLE design)
At the start: 86.4 x 31.8 mm, 84 parts, among them IC1 STM32F051C6T, J3 CONN_PWM, J4 TEMP_DO, J5 CONN_FAN, J6 CONN_I2C, J7 EC, P1 KF128-2P, Q1 600mA/40V, U1 BL9341, U2 BL9341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

Commit message: 调整敷铜
Routing:
- net GND: vias 81 -> 87
Changed lines of the file:
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@@
 <via x="26.67" y="16.51" extent="1-16" drill="0.3"/>
 <via x="31.75" y="16.637" extent="1-16" drill="0.3"/>
-<via x="29.21" y="13.97" extent="1-16" drill="0.3"/>
+<via x="31.242" y="13.081" extent="1-16" drill="0.3"/>
 <via x="36.83" y="21.59" extent="1-16" drill="0.3"/>
 <via x="36.83" y="25.4" extent="1-16" drill="0.3"/>
@@
 <via x="60.96" y="24.13" extent="1-16" drill="0.3"/>
 <contactref element="J4" pad="3"/>
+<via x="31.242" y="4.445" extent="1-16" drill="0.3"/>
+<via x="31.242" y="6.985" extent="1-16" drill="0.3"/>
+<via x="29.21" y="13.97" extent="1-16" drill="0.3"/>
+<via x="49.53" y="5.08" extent="1-16" drill="0.3"/>
+<via x="53.34" y="2.54" extent="1-16" drill="0.3"/>
+<via x="37.973" y="0.762" extent="1-16" drill="0.3"/>
 </signal>
 <signal name="N$1">
@@
 <contactref element="IC1" pad="7"/>
 <contactref element="S1" pad="1"/>
-<wire x1="44.958" y1="7.887" x2="42.025" y2="7.887" width="0.254" layer="1"/>
+<wire x1="44.958" y1="7.887" x2="42.037" y2="7.887" width="0.254" layer="1"/>
+<wire x1="42.037" y1="7.887" x2="42.025" y2="7.887" width="0.254" layer="1"/>
 <wire x1="42.025" y1="7.887" x2="41.91" y2="7.772" width="0.254" layer="1"/>
 <wire x1="44.958" y1="7.887" x2="44.958" y2="9.131" width="0.254" layer="1"/>
@@
 <wire x1="22.225" y1="8.128" x2="24.13" y2="8.128" width="0.254" layer="16"/>
 <wire x1="24.13" y1="8.128" x2="25.527" y2="9.525" width="0.254" layer="16"/>
-<wire x1="37.846" y1="9.525" x2="39.497" y2="7.874" width="0.254" layer="16"/>
 <wire x1="25.527" y1="9.525" x2="30.8666375" y2="9.525" width="0.254" layer="16"/>
-<wire x1="30.8666375" y1="9.525" x2="37.846" y2="9.525" width="0.254" layer="16"/>
-<via x="39.497" y="7.874" extent="1-16" drill="0.3"/>
-<wire x1="39.497" y1="7.874" x2="41.808" y2="7.874" width="0.254" layer="1"/>
-<wire x1="41.808" y1="7.874" x2="41.91" y2="7.772" width="0.254" layer="1"/>
+<wire x1="30.8666375" y1="9.525" x2="39.497" y2="9.525" width="0.254" layer="16"/>
+<via x="39.497" y="9.525" extent="1-16" drill="0.3"/>
 <wire x1="21.717" y1="7.62" x2="22.225" y2="8.128" width="0.254" layer="16"/>
+<wire x1="39.497" y1="9.525" x2="40.399" y2="9.525" width="0.254" layer="1"/>
+<wire x1="40.399" y1="9.525" x2="42.037" y2="7.887" width="0.254" layer="1"/>
 </signal>
 <signal name="TX">

Commit message: 调整敷铜
Routing:
- net EC_B: track 30.2 -> 27.8 mm
- net GND: vias 87 -> 88
Changed lines of the file:
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@@
 <via x="53.34" y="2.54" extent="1-16" drill="0.3"/>
 <via x="37.973" y="0.762" extent="1-16" drill="0.3"/>
+<via x="18.923" y="7.112" extent="1-16" drill="0.3"/>
 </signal>
 <signal name="N$1">
@@
 <wire x1="29.21" y1="22.365" x2="29.21" y2="25.21" width="0.254" layer="1"/>
 <wire x1="29.21" y1="25.21" x2="29.4" y2="25.4" width="0.254" layer="1"/>
-<wire x1="17.554" y1="3.624" x2="17.554" y2="2.893" width="0.254" layer="1"/>
-<wire x1="17.554" y1="2.893" x2="18.034" y2="2.413" width="0.254" layer="1"/>
-<via x="18.034" y="2.413" extent="1-16" drill="0.3"/>
-<wire x1="18.034" y1="2.413" x2="18.034" y2="13.081" width="0.254" layer="16"/>
+<via x="18.034" y="6.096" extent="1-16" drill="0.3"/>
+<wire x1="18.034" y1="6.096" x2="18.034" y2="13.081" width="0.254" layer="16"/>
 <wire x1="18.034" y1="13.081" x2="26.543" y2="21.59" width="0.254" layer="16"/>
 <via x="26.543" y="21.59" extent="1-16" drill="0.3"/>
 <wire x1="26.543" y1="21.59" x2="27.318" y2="22.365" width="0.254" layer="1"/>
 <wire x1="27.318" y1="22.365" x2="27.686" y2="22.365" width="0.254" layer="1"/>
+<wire x1="17.554" y1="3.624" x2="17.554" y2="4.727" width="0.254" layer="1"/>
+<wire x1="17.554" y1="4.727" x2="18.034" y2="5.207" width="0.254" layer="1"/>
+<wire x1="18.034" y1="5.207" x2="18.034" y2="6.096" width="0.254" layer="1"/>
 </signal>
 <signal name="EC_A">
